File: PCB/leds_controller.kicad_pcb (KiCad board)
At the start: 2 copper layers, 46 x 31 mm, 26 parts, among them J1 Barrel_Jack, U0 STM8S001J3M, U1 MC78M05_TO252

Commit message: updating to kicad 10, including 3D models screenshots
Connections:
- J1 pad 3: GND -> (no net)

Commit message: updated doc
Parts:
- C1: value C -> 100n
- CVCAP1: value C -> 1u
- R1, R10, R2, R3: value R -> 1k
- R11, R4, R5, R6: value R -> 47k
- R7, R8, R9: value R -> 560
Changed lines of the file:
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@@
 			)
 		)
-		(property "Value" "C"
+		(property "Value" "1u"
 			(at 0 1.43 0)
 			(layer "F.Fab")
@@
 			)
 		)
-		(property "Value" "C"
+		(property "Value" "100n"
 			(at 0 1.43 90)
 			(layer "F.Fab")
@@
 			)
 		)
-		(property "Value" "R"
+		(property "Value" "560"
 			(at 0 1.43 0)
 			(layer "F.Fab")
@@
 			)
 		)
-		(property "Value" "R"
+		(property "Value" "1k"
 			(at 0 1.43 90)
 			(layer "F.Fab")
@@
 			)
 		)
-		(property "Value" "R"
+		(property "Value" "1k"
 			(at 0 1.43 90)
 			(layer "F.Fab")
@@
 			)
 		)
-		(property "Value" "R"
+		(property "Value" "1k"
 			(at 0 1.43 0)
 			(layer "F.Fab")
@@
 			)
 		)
-		(property "Value" "R"
+		(property "Value" "47k"
 			(at 0 1.43 0)
 			(layer "F.Fab")
@@
 			)
 		)
-		(property "Value" "R"
+		(property "Value" "47k"
 			(at 0 1.43 0)
 			(layer "F.Fab")
@@
 			)
 		)
-		(property "Value" "R"
+		(property "Value" "47k"
 			(at 0 1.43 0)
 			(layer "F.Fab")
@@
 			)
 		)
-		(property "Value" "R"
+		(property "Value" "1k"
 			(at 0 1.43 90)
 			(layer "F.Fab")
@@
 			)
 		)
-		(property "Value" "R"
+		(property "Value" "560"
 			(at 0 1.43 0)
 			(layer "F.Fab")
@@
 			)
 		)
-		(property "Value" "R"
+		(property "Value" "47k"
 			(at 0 1.43 0)
 			(layer "F.Fab")
@@
 			)
 		)
-		(property "Value" "R"
+		(property "Value" "560"
 			(at 0 1.43 0)
 			(layer "F.Fab")
